File: Projet_Bagnole.sch (KiCad schematic (older format))
At the start: 50 parts, among them J1 USB_A, J2 Conn_01x03_Male, J3 Conn_01x04_Male, J4 AVR-ISP-6, M1 Motor_DC, M2 Stepper_Motor_bipolar, U1 ATmega16U2-AU, U2 DRV8210DRL, U3 MAX1811, Y1 Crystal_GND24

Commit message: V2
Parts:
- added ANT?: ANT3216LL00R2400A, symbol Projet_Bagnole-rescue:ANT3216LL00R2400A
- added C? (x2): C, symbol Device:C
- added C? (x2): 10uF, symbol Device:C
- added L?: L, symbol Device:L
- added R?: 4.7k, symbol Device:R
- added U?: BM71BLE01FC2, symbol Projet_Bagnole-rescue:BM71BLE01FC2
- M1: footprint (none) -> Connector_PinHeader_2.54mm:PinHeader_1x02_P2.54mm_Vertical
- M2: footprint (none) -> Connector_PinHeader_2.54mm:PinHeader_2x02_P2.54mm_Vertical
Connections:
- net GND: now also C?.1, C?.2, C?.2, C?.2, U?.12 (GND), U?.17 (GND)
- net VCC: now also C?.2, R?.1, U?.10 (BK_IN)
- new net: ANT?.1 (FEEDING), C?.1, L?.2
- new net ANTENNE: C?.1, L?.1, U?.1 (BT_RF)
- new net RST_N: C?.1, R?.2, U?.7 (RST__N)
- new net SOLDERING: ANT?.2 (SOLDERING)
Other:
- moved on the sheet: C1, C10, C2, C3, C4, C5, C6, C7, C8, C9, D1, D13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

Commit message: V3
Parts:
- added R19: R, Resistor_SMD:R_0603_1608Metric, symbol Device:R
- added U5: LM4040DBZ-2.5, Package_TO_SOT_SMD:SOT-23, symbol Reference_Voltage:LM4040DBZ-2.5
- ANT1: renamed from ANT?; footprint (none) -> Projet_Bagnole:ANT3216LL00R2400A
- C11, C12, C13, C14: renamed from C?; footprint (none) -> Capacitor_SMD:C_0603_1608Metric
- L1: renamed from L?; footprint (none) -> Inductor_SMD:L_0603_1608Metric
- M1: footprint Connector_PinHeader_2.54mm:PinHeader_1x02_P2.54mm_Vertical -> Projet_Bagnole:Motor_DC
- M2: footprint Connector_PinHeader_2.54mm:PinHeader_2x02_P2.54mm_Vertical -> Projet_Bagnole:Motor_Prop
- R18: renamed from R?; footprint (none) -> Resistor_SMD:R_0603_1608Metric
- U4: renamed from U?; footprint (none) -> Projet_Bagnole:BM71BLE01FC2
Connections:
- net GND: now also U5.2 (A)
- net VCC: now also R19.1; no longer C13.2, U4.10 (BK_IN)
- net 2.5V: now reaches U4.11 (VBAT)
- net 2.5V: now also C13.2, U4.10 (BK_IN), R19.2, U5.1 (K)
Other:
- moved on the sheet: ANT1, C11, C12, C13, C14, L1, R18, U4

Commit message: 04/04 -Routage presque terminé
Parts:
- J2: footprint Connector_PinHeader_2.54mm:PinHeader_1x03_P2.54mm_Vertical -> Connector_Molex:Molex_PicoBlade_53048-0310_1x03_P1.25mm_Horizontal
- M2: footprint Projet_Bagnole:Motor_Prop -> rex-motors:micro-slider
Changed lines of the file:
@@
 F 0 "M2" H 10288 1124 50  0000 L CNN
 F 1 "Stepper_Motor_bipolar" H 10288 1033 50  0000 L CNN
-F 2 "Projet_Bagnole:Motor_Prop" H 10110 990 50  0001 C CNN
+F 2 "rex-motors:micro-slider" H 10110 990 50  0001 C CNN
 F 3 "http://www.infineon.com/dgdl/Application-Note-TLE8110EE_driving_UniPolarStepperMotor_V1.1.pdf?fileId=db3a30431be39b97011be5d0aa0a00b0" H 10110 990 50  0001 C CNN
 	1    10100 1000
@@
 F 0 "J2" H 6172 5732 50  0000 R CNN
 F 1 "Conn_01x03_Male" H 6172 5823 50  0000 R CNN
-F 2 "Connector_PinHeader_2.54mm:PinHeader_1x03_P2.54mm_Vertical" H 6200 5800 50  0001 C CNN
+F 2 "Connector_Molex:Molex_PicoBlade_53048-0310_1x03_P1.25mm_Horizontal" H 6200 5800 50  0001 C CNN
 F 3 "~" H 6200 5800 50  0001 C CNN
 	1    6200 5800
